File: pcb/AmplificadorV2/AmplificadorV2/AmplificadorV2.sch (KiCad schematic (older format))
At the start: 16 parts

Commit message: new ampli in progress
Parts:
- removed C? (x16): C, symbol Device:C
- added C1: C, FootprintAmpli:QFN40P700X700X75-61N, symbol Device:C
- added C10, C11, C12, C13, C14, C15, C2, C3, C5, C7, C8, C9: C, symbol Device:C
- added C4: 0.1uF, symbol Device:C
- added C6: 5.6pF, symbol Device:C
- added J1, J2, J3, J4, J5, Vg2: Conn_01x01_Female, symbol Connector:Conn_01x01_Female
- added R1: 4.7K, symbol Device:R
- added R2: 4.7k, symbol Device:R
- added U1: MHT2012N, FootprintAmpli:QFN-24_EP_8x8_Pitch0.8mm, symbol AmplifierRaul:MHT2012N
Connections:
- new net: C1.1, C4.1, C6.1, R1.1, U1.8 (VGS2)
- new net: R1.2, Vg2.1 (Pin_1)
- new net: C2.1, C3.1, C5.1, C7.1, R2.1
- new net: J2.1 (Pin_1), R2.2
- new net: C12.1, C14.1, C15.1, C9.1, J5.1 (Pin_1), U1.10 (VDS1)
- new net: C10.1, C11.1, C13.1, C8.1, J3.1 (Pin_1), J4.1 (Pin_1), U1.15 (RFout/VDS2), U1.16 (RFout/VDS2)
- new net: C7.2, U1.24 (Vgs1)
- new net: J1.1 (Pin_1), U1.3 (Rfin), U1.4 (RFin)
- new net GND: C1.2, C10.2, C11.2, C12.2, C13.2, C14.2, C15.2, C2.2, C3.2, C4.2, C5.2, C6.2, C8.2, C9.2
