File: pcb/AmplificadorV2/AmplificadorV2/AmplificadorV2.sch (KiCad schematic (older format))
At the start: 28 parts, among them J1 Conn_01x01_Female, J2 Conn_01x01_Female, J3 Conn_01x01_Female, J4 Conn_01x01_Female, J5 Conn_01x01_Female, U1 MHT2012N

Commit message: avances
Connections:
- net labels added: condensador
Changed lines of the file:
@@
 	8550 6000 8550 5550
-Wire Wire Line
-	8050 5550 7950 5550
 Wire Wire Line
 	6450 5550 7250 5550
@@
 Text GLabel 7000 4900 1    50   Input ~ 0
 outAmpli
+Wire Wire Line
+	7950 5550 8550 5550
+Text GLabel 8050 4000 1    50   Input ~ 0
+condensador
 $EndSCHEMATC
